File: hardware/mek-core-ctrl/power.kicad_sch (KiCad schematic)
At the start: 22 parts, among them J1 24-26VAC, U1 LMR38020FDDAR, U2 AMS1117-3.3

Commit message: Creating mek-output-expander
Parts:
- R1: footprint (none) -> Resistor_SMD:R_1206_3216Metric
Changed lines of the file:
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@@
 			)
 		)
-		(property "Footprint" ""
+		(property "Footprint" "Resistor_SMD:R_1206_3216Metric"
 			(at 52.07 104.14 0)
 			(hide yes)
