File: hardware/triac_fet_module/triac_fet_module.kicad_sch (KiCad schematic)
At the start: 13 parts, among them J1 Conn_01x02_Pin, J2 Screw_Terminal_01x02, Q1 BT136-800, U1 MOC3063M

Commit message: Creating mek-output-expander
Parts:
- U1: footprint Package_SO:TSOP-6_1.65x3.05mm_P0.95mm -> Package_DIP:SMDIP-6_W9.53mm
Changed lines of the file:
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@@
 			)
 		)
-		(property "Footprint" "Package_SO:TSOP-6_1.65x3.05mm_P0.95mm"
+		(property "Footprint" "Package_DIP:SMDIP-6_W9.53mm"
 			(at 148.59 91.44 0)
 			(hide yes)
