File: hardware/mek-sub-triac/mek-sub-triac.kicad_sch (KiCad schematic)
At the start: 21 parts, among them J1 Conn_01x04_Pin, J2 Screw_Terminal_01x02, Q1 MMBT3904, Q2 BT136S-800E, U1 MOC3063S

Commit message: Initial PCB layout
Parts:
- removed C2: 100n, Mekatrol:C_0603_1206_Combo_Paste0603, symbol Device:C_Small
- added H2: MountingHole_Pad, MountingHole:MountingHole_2.7mm, symbol Mechanical:MountingHole
- C1: footprint Mekatrol:C_0603_1206_Combo_Paste0603 -> Capacitor_SMD:C_1206_3216Metric
- D1: footprint Mekatrol:D_0603_1206_Combo_Diode_Paste0603 -> LED_SMD:LED_0805_2012Metric
- H1: footprint MountingHole:MountingHole_3.2mm_M3_Pad_Via -> MountingHole:MountingHole_2.7mm; symbol Mechanical:MountingHole_Pad -> Mechanical:MountingHole
- R1, R2, R6: footprint Mekatrol:R_0603_1206_Combo_Paste0603 -> Resistor_SMD:R_1206_3216Metric
- R3, R4, R5: footprint Mekatrol:R_0603_1206_Combo_Paste0603 -> Resistor_SMD:R_0603_1608Metric
- R7: footprint Mekatrol:R_0603_1206_Combo_Paste0603 -> Resistor_SMD:R_2512_6332Metric
- renumbered C3 to C2
Connections:
- net GND: no longer H1.1
- net MT2_FB: now reaches R5.1, U1.6
- net MT2: now reaches D2.2 (A2), J2.2 (Pin_2), Q2.2 (A2), R5.2, R7.2
- net MT1_FB: now reaches Q2.3 (G), R6.1, U1.4
- net MT1: now reaches C2.2, D2.1 (A1), J2.1 (Pin_1), Q2.1 (A1), R6.2
- net +3V3: no longer names the net of J1.2 (Pin_2)
- no-connect marks 0 -> 1
